File: KiCad/QuinoaChipPlant.kicad_pcb (KiCad board)
At the start: 2 copper layers, 195.3 x 185 mm, 104 parts, among them J1 GROVE, J10 BULB, J11 LEVEL2, J12 LEVEL3, J13 LEVEL4, J15 BULB, J16 BULB, J18 GROVE, J2 DCJACK, J3 LEVEL1, J4 Screw_Terminal_01x03, J5 MOTOR, J6 MOTOR, J7 BULB, J8 BULB, J9 BULB, SW1 SW_Push, U1 ESP32_DEVKIT_V1, U2 SparkFun_TB6612FNG_MOTOR_DRIV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, U3 SparkFun_TB6612FNG_MOTOR_DRIV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, U4 SparkFun_TB6612FNG_MOTOR_DRIV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, U5 SEEED_GROVE, U7 CR2013-MI2120

Commit message: Ver.20230911
Parts:
- removed R2: 470, Resistor_SMD:R_1206_3216Metric_Pad1.30x1.75mm_HandSolder
- removed REF** (x4): MountingHole_3.2mm_M3, MountingHole:MountingHole_3.2mm_M3
- added C12: C, Resistor_SMD:R_1206_3216Metric_Pad1.30x1.75mm_HandSolder, F.Cu at (232.8, 206.2)
- added C13: C, Resistor_SMD:R_1206_3216Metric_Pad1.30x1.75mm_HandSolder, F.Cu at (337.6, 199.9)
- added C14: C, Resistor_SMD:R_1206_3216Metric_Pad1.30x1.75mm_HandSolder, F.Cu at (291.4, 350.5)
- added C15: C_Polarized, Capacitor_THT:CP_Radial_D10.0mm_P2.50mm_P5.00mm, F.Cu at (297.2, 343.5)
- added C16: C, Resistor_SMD:R_1206_3216Metric_Pad1.30x1.75mm_HandSolder, F.Cu at (366.8, 142.8)
- added C17: C, Resistor_SMD:R_1206_3216Metric_Pad1.30x1.75mm_HandSolder, F.Cu at (366.9, 129.2)
- added D10: D, Diode_SMD:D_SOD-123, F.Cu at (236.0, 219.8)
- added D11: D, Diode_SMD:D_SOD-123, F.Cu at (340.2, 212.6)
- added D12: LED, LED_THT:LED_D3.0mm, F.Cu at (230.1, 221.1)
- added D13: LED, LED_THT:LED_D3.0mm, F.Cu at (335.7, 213.8)
- added D14: LED, LED_THT:LED_D3.0mm, F.Cu at (334.8, 178.2)
- added D15: LED, LED_THT:LED_D3.0mm, F.Cu at (345.1, 178.3)
- added D16: LED, LED_THT:LED_D3.0mm, F.Cu at (355.0, 178.5)
- added D17: LED, LED_THT:LED_D3.0mm, F.Cu at (364.5, 178.5)
- added D18: D, Diode_SMD:D_SOD-123, F.Cu at (369.0, 133.3)
- added D19: LED, LED_THT:LED_D3.0mm, F.Cu at (364.9, 149.2)
- added D20: LED, LED_THT:LED_D3.0mm, F.Cu at (364.9, 134.6)
- added D8: LED, LED_THT:LED_D3.0mm, F.Cu at (227.0, 290.0)
- added D9: LED, LED_THT:LED_D3.0mm, F.Cu at (337.0, 286.0)
- added J14: DCJACK OPTIONAL, library:DCJACK, F.Cu at (293.0, 372.0)
- added J20: Screw_Terminal_01x04, TerminalBlock_Phoenix:TerminalBlock_Phoenix_PT-1,5-4-5.0-H_1x04_P5.00mm_Horizontal, F.Cu at (366.1, 125.0)
- added JP2: SolderJumper_2_Bridged, Jumper:SolderJumper-2_P1.3mm_Bridged_Pad1.0x1.5mm, F.Cu at (283.6, 354.5)
- added JP3: SolderJumper_2_Bridged, Jumper:SolderJumper-2_P1.3mm_Bridged_Pad1.0x1.5mm, F.Cu at (289.8, 359.2)
- added R11: 470, Resistor_SMD:R_1206_3216Metric_Pad1.30x1.75mm_HandSolder, F.Cu at (228.6, 294.0)
- added R12: 470, Resistor_SMD:R_1206_3216Metric_Pad1.30x1.75mm_HandSolder, F.Cu at (341.6, 289.0)
- added R13: 470, Resistor_SMD:R_1206_3216Metric_Pad1.30x1.75mm_HandSolder, F.Cu at (232.9, 225.0)
- added R14: 470, Resistor_SMD:R_1206_3216Metric_Pad1.30x1.75mm_HandSolder, F.Cu at (337.4, 218.5)
- added R15: 470, Resistor_SMD:R_1206_3216Metric_Pad1.30x1.75mm_HandSolder, F.Cu at (336.9, 182.0)
- added R16: 470, Resistor_SMD:R_1206_3216Metric_Pad1.30x1.75mm_HandSolder, F.Cu at (347.8, 182.0)
- added R17: 470, Resistor_SMD:R_1206_3216Metric_Pad1.30x1.75mm_HandSolder, F.Cu at (356.6, 182.5)
- added R18: 470, Resistor_SMD:R_1206_3216Metric_Pad1.30x1.75mm_HandSolder, F.Cu at (365.9, 182.5)
- added R19: 470, Resistor_SMD:R_1206_3216Metric_Pad1.30x1.75mm_HandSolder, F.Cu at (366.9, 153.0)
- added R20: 470, Resistor_SMD:R_1206_3216Metric_Pad1.30x1.75mm_HandSolder, F.Cu at (366.9, 138.0)
- added REF07: MountingHole_4.3mm_M4_DIN965, MountingHole:MountingHole_4.3mm_M4_DIN965, F.Cu at (357.0, 148.0)
- added REF09: MountingHole_4.3mm_M4_DIN965, MountingHole:MountingHole_4.3mm_M4_DIN965, F.Cu at (338.0, 90.0)
- added U6: SparkFun_TB6612FNG_MOTOR_DRIVER_MODULE, library:SparkFun_TB6612FNG_MOTOR_DRIVER_MODULE, F.Cu at (354.6, 273.9)
- added U8: SparkFun_TB6612FNG_MOTOR_DRIVER_MODULE, library:SparkFun_TB6612FNG_MOTOR_DRIVER_MODULE, F.Cu at (354.6, 204.1)
- C10, C11, C6, C7, C8, C9: footprint Capacitor_THT:CP_Radial_D5.0mm_P2.00mm -> Resistor_SMD:R_1206_3216Metric_Pad1.30x1.75mm_HandSolder
- D1: value LED -> D; footprint LED_THT:LED_D3.0mm -> Diode_SMD:D_SOD-123
- D2, D3, D4, D5, D6, D7: footprint Diode_THT:D_DO-41_SOD81_P5.08mm_Vertical_KathodeUp -> Diode_SMD:D_SOD-123
- J4: value Screw_Terminal_01x03 -> Screw_Terminal_01x04; footprint TerminalBlock_Philmore:TerminalBlock_Philmore_TB133_1x03_P5.00mm_Horizontal -> TerminalBlock_Phoenix:TerminalBlock_Phoenix_PT-1,5-4-5.0-H_1x04_P5.00mm_Horizontal
- moved REF12 318.7 mm to (366.0, 372.5), turned to -90 degrees
- moved J3 310.7 mm to (367.6, 344.0), turned to 180 degrees
- moved TH1 305.6 mm to (363.5, 351.2), turned to -90 degrees
- moved J11 292.3 mm to (367.5, 334.0), turned to 180 degrees
- moved U5 281.4 mm to (365.0, 364.5)
- moved J18 281.3 mm to (338.0, 361.0)
- moved J12 274.9 mm to (367.8, 324.0), turned to 180 degrees
- moved J1 273.0 mm to (334.8, 343.0)
- moved U1 270.3 mm to (339.7, 344.9), turned to 90 degrees
- moved REF08 264.0 mm to (366.0, 90.0), turned to -90 degrees
- moved R1 264.0 mm to (350.9, 326.0)
- moved J2 261.8 mm to (274.0, 372.0), turned to 90 degrees
- moved R7 258.2 mm to (352.4, 321.5)
- moved J13 256.8 mm to (367.8, 314.0), turned to 180 degrees
- moved R8 251.5 mm to (352.6, 317.5), turned to 180 degrees
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- renumbered REF** to REF08, REF** to REF10, REF** to REF100, REF** to REF11, REF** to REF111, REF** to REF112, REF** to REF113, REF** to REF114, REF** to REF115, REF** to REF116, REF** to REF117, REF** to REF118, REF** to REF119, REF** to REF12, REF** to REF120, REF** to REF121, REF** to REF122, REF** to REF123, REF** to REF124, REF** to REF125, REF** to REF126, REF** to REF127, REF** to REF128, REF** to REF129, REF** to REF13, REF** to REF130, REF** to REF131, REF** to REF132, REF** to REF133, REF** to REF134, REF** to REF14, REF** to REF140, REF** to REF141, REF** to REF15, REF** to REF16, REF** to REF17, REF** to REF18, REF** to REF19, REF** to REF21, REF** to REF22, REF** to REF23, REF** to REF230, REF** to REF24, REF** to REF26, REF** to REF27
Connections:
- C1 pad 1: Vdrive -> +12V
- C2 pad 1: Vdrive -> +12V
- C3 pad 1: +5V -> +12VA
- C4 pad 1: +5V -> +12VA
- D1 pad 1: WATERSENSOR1 -> Net-(D1-K)
- J2 pad 1: +5V -> +12V
- J4 pad 1: Vdrive -> VDDA
- J4 pad 2: +5V -> +12V
- J4 pad 3: GND -> +12VA
- J5 pad 1: Net-(D2-K) -> Net-(D2-A)
- J5 pad 2: Net-(D2-A) -> Net-(D2-K)
- J6 pad 1: Net-(D3-K) -> Net-(D3-A)
- J6 pad 2: Net-(D3-A) -> Net-(D3-K)
- J7 pad 1: Net-(D2-A) -> Net-(D10-A)
- J7 pad 2: Net-(D2-K) -> Net-(D10-K)
- J8 pad 1: Net-(D3-A) -> Net-(D11-A)
- J8 pad 2: Net-(D3-K) -> Net-(D11-K)
- JP1 pad 1: +5V -> +12V
- JP1 pad 2: Vdrive -> VDDA
- U1 pad 12: unconnected-(U1-Pad12) -> RELAY1
- U1 pad 15: +5V -> VDDA
- U1 pad 18: unconnected-(U1-15-Pad18) -> WATERSENSOR4
- U1 pad 7: WATERSENSOR4 -> RELAY2
- U2 pad 1: Vdrive -> +12VA
- U2 pad 11: +3V3 -> GND
- U3 pad 1: Vdrive -> +12V
- U3 pad 11: +3V3 -> GND
- U4 pad 1: Vdrive -> +12V
- U4 pad 11: +3V3 -> GND
Routing:
- net +12V: track 0.00 -> 329.5 mm, vias 0 -> 4
- net GND: track 257.3 -> 505.7 mm, vias 2 -> 11
- net Vdrive: track 235.6 -> 20.4 mm, vias 3 -> 0
- net Net-(D10-A): track 0.00 -> 197.1 mm, vias 0 -> 2
- net +12VA: track 0.00 -> 196.2 mm, vias 0 -> 1
- net Net-(D10-K): track 0.00 -> 186.7 mm, vias 0 -> 1
- net RELAY2: track 0.00 -> 166.6 mm, vias 0 -> 2
- net Net-(D18-A): track 0.00 -> 152.1 mm
- net RELAY1: track 0.00 -> 148.7 mm
- net VDDA: track 0.00 -> 146.0 mm, vias 0 -> 3
- net Net-(U1-5): track 157.4 -> 11.6 mm
- net Net-(D18-K): track 0.00 -> 144.8 mm, vias 0 -> 1
- net Net-(U1-4): track 150.8 -> 6.27 mm, vias 1 -> 0
- net Net-(U1-18): track 156.7 -> 12.7 mm
- net Net-(U1-17): track 151.2 -> 7.32 mm, vias 1 -> 0
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- added copper zone on F.Cu, net GND
- removed copper zone on F.Cu, net +5V
Other:
- board size 195.3 x 185 mm -> 148.5 x 293 mm
- board text added: "0.1uF x 3"
- board text added: "1"
- board text added: "10k (thermistor)"
- board text added: "10k x 4"
- board text added: "2"
- board text added: "3"
- board text added: "4"
- board text added: "470 x 4"
- board text added: "ELLIPSE HOLE x 9"
- board text added: "QuinoaChipPlant Robot Ver.20230911 https://github.com/nanbuwks/QuinoaChipPlant"
- board text added: "VIN 12V 12VA GND"
- board text added: "バルブ"
- board text added: "ポンプ1 給水"
- board text added: "ポンプ2 排水"
- board text removed: "5V Cx2"
- board text removed: "GND"
- board text removed: "MOTOR DRIVER"
- board text removed: "QuinoaChipPlant Water Control Ver.20230579 https://github.com/nanbuwks/QuinoaChipPlant"
- board text removed: "VDRIVE"
- board text removed: "VDRIVE 5V GND"
- board text removed: "VDRIVE Cx2"
- board text removed: "VDrive 5V GND"

Commit message: 202311 version
Parts:
- removed JP1, JP2: SolderJumper_2_Bridged, Jumper:SolderJumper-2_P1.3mm_Bridged_Pad1.0x1.5mm
- added ?: , , F.Cu at (335.5, 170.5)
- added ?: , , F.Cu at (346.5, 319.5)
- added ?: , , F.Cu at (346.5, 316.5)
- added ?: , , F.Cu at (342.0, 211.5)
- added ?: , , F.Cu at (335.5, 173.5)
- added ?: , , F.Cu at (335.5, 167.5)
- added ?: , , F.Cu at (346.5, 249.0)
- added ?: , , F.Cu at (346.5, 252.5)
- added REF**: SeparateHole, MountingHole:MountingHole_2.1mm, F.Cu at (335.0, 122.0)
- added REF**: SeparateHole, MountingHole:MountingHole_2.1mm, F.Cu at (335.0, 119.0)
- added REF**: SeparateHole, MountingHole:MountingHole_2.1mm, F.Cu at (335.0, 126.0)
- added REF**: SeparateHole, MountingHole:MountingHole_2.1mm, F.Cu at (335.5, 94.5)
- added REF08: MountingHole_3.2mm_M3, MountingHole:MountingHole_3.2mm_M3, F.Cu at (401.0, 95.0)
- added REF12: MountingHole_3.2mm_M3, MountingHole:MountingHole_3.2mm_M3, F.Cu at (398.5, 334.5)
- added REF12: MountingHole_3.2mm_M3, MountingHole:MountingHole_3.2mm_M3, F.Cu at (353.5, 334.0)
- added U9: ~, library:YRB_YMD-10WR3_YRA_YMD-10WR3, F.Cu at (375.4, 266.7)
- TH1: footprint TerminalBlock:TerminalBlock_Altech_AK300-2_P5.00mm -> TerminalBlock_Phoenix:TerminalBlock_Phoenix_MKDS-1,5-2_1x02_P5.00mm_Horizontal
- moved J4 214.8 mm to (398.2, 216.5), turned to 90 degrees
- moved JP3 182.7 mm to (383.6, 202.5)
- moved J14 181.3 mm to (400.5, 226.0), turned to 180 degrees
- moved J2 180.5 mm to (400.3, 242.9), turned to 180 degrees
- moved C1 180.4 mm to (378.8, 201.1), turned to 90 degrees
- moved SW1 179.5 mm to (402.2, 328.8), turned to 180 degrees
- moved C2 170.8 mm to (378.9, 210.7)
- moved C3 168.0 mm to (385.3, 215.9), turned to -90 degrees
- moved C4 154.2 mm to (378.9, 221.7)
- moved R11 143.3 mm to (355.9, 228.3)
- moved D8 142.8 mm to (354.5, 225.6)
- moved D2 141.9 mm to (358.5, 224.5)
- moved J5 141.8 mm to (356.5, 216.3), turned to -90 degrees
- moved C6 138.6 mm to (356.4, 212.0)
- moved BZ1 132.5 mm to (362.0, 324.0), turned to 180 degrees
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Connections:
- C14 pad 1: VDDA -> +5V
- C15 pad 1: VDDA -> +5V
- J1 pad 3: Vdrive -> +5V
- J18 pad 3: Vdrive -> +5V
- J4 pad 1: VDDA -> +5V
- U1 pad 15: VDDA -> +5V
Routing:
- net GND: track 505.7 -> 821.6 mm, vias 11 -> 10
- net +5V: track 0.00 -> 198.3 mm, vias 0 -> 2
- net VDDA: track 146.0 -> 0.00 mm, vias 3 -> 0
- net Net-(BZ1--): track 163.3 -> 23.6 mm, vias 1 -> 0
- net SW_THERMISTOR: track 205.8 -> 76.8 mm, vias 3 -> 1
- net Net-(D10-A): track 197.1 -> 69.7 mm, vias 2 -> 1
- net Net-(D10-K): track 186.7 -> 75.9 mm
- net Net-(D18-K): track 144.8 -> 38.5 mm, vias 1 -> 0
- net +12VA: track 196.2 -> 92.0 mm, vias 1 -> 2
- net MOTOR1: track 126.5 -> 224.8 mm
- net Net-(U1-5): track 11.6 -> 109.7 mm, vias 0 -> 1
- net Net-(U1-23): track 26.6 -> 124.2 mm
- net Net-(U1-17): track 7.32 -> 104.2 mm, vias 0 -> 1
- net Net-(U1-18): track 12.7 -> 106.0 mm
- net Net-(U1-16): track 11.9 -> 102.1 mm
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- added copper zone on B.Cu, net (none)
- added copper zone on F.Cu, net (none)
- removed copper zone on B.Cu, net GND
- removed copper zone on F.Cu, net GND
Other:
- board size 148.5 x 293 mm -> 180 x 263.2 mm
- board text added: "5V 12V MOTOR GND"
- board text added: "ELLIPSE HOLE x 14"
- board text added: "QuinoaChipPlant Robot Ver.20231022 https://github.com/nanbuwks/QuinoaChipPlant"
- board text removed: "470 x 4"
- board text removed: "ELLIPSE HOLE x 9"
- board text removed: "QuinoaChipPlant Robot Ver.20230911 https://github.com/nanbuwks/QuinoaChipPlant"
- board text removed: "VIN 12V 12VA GND"
