File: KiCad/QuinoaChipPlant.kicad_sch (KiCad schematic)
At the start: 88 parts, among them J1 GROVE, J10 BULB, J11 LEVEL2, J12 LEVEL3, J13 LEVEL4, J14 DCJACK OPTIONAL, J15 BULB, J16 BULB, J18 GROVE, J2 DCJACK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

Commit message: 202311 version
Parts:
- removed JP1, JP2: SolderJumper_2_Bridged, Jumper:SolderJumper-2_P1.3mm_Bridged_Pad1.0x1.5mm, symbol Jumper:SolderJumper_2_Bridged
- added U9: ~, library:YRB_YMD-10WR3_YRA_YMD-10WR3, symbol nanbuwks:VRB_YMD-10WR3_VRA_YMD-10WR3
- TH1: footprint TerminalBlock:TerminalBlock_Altech_AK300-2_P5.00mm -> TerminalBlock_Phoenix:TerminalBlock_Phoenix_MKDS-1,5-2_1x02_P5.00mm_Horizontal
Connections:
- net VDDA is gone; now on net +5V: C14.1, C15.1, J4.1 (Pin_1), U1.15 (VIN)
- net Vdrive is gone; now on net +5V: J1.3 (Pin_3), J18.3 (Pin_3)
- net +12V: now also U9.1 (-Vin)
- net +5V: now also U9.3 (+Vo)
- net GND: now also U9.2 (+Vin), U9.5 (0V/-Vo)
- no-connect marks 7 -> 8
Other:
- moved on the sheet: C1, C14, C15, C2, C3, C4, J14, J2, J4, JP3, U1
